File: display.kicad_sch (KiCad schematic)
At the start: 12 parts, among them IC13 LSF0204GU12X, J3 505110-1492, J4 SM02B-SRSS-TB_LF__SN_

Commit message: Add company name (using github URL), date, and change revision number to all schematic pages
Other:
- company: (none) -> github.com/fuad1502/open-running-watch-hw
Changed lines of the file:
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@@
 	(title_block
 		(title "Open Running Watch")
-		(rev "A")
+		(date "2024-04-12")
+		(rev "0.1.0")
+		(company "github.com/fuad1502/open-running-watch-hw")
 	)
 	(junction
