File: bluenrg.kicad_sch (KiCad schematic)
At the start: 24 parts, among them IC1 BLUENRG-232N, T1 BALF-NRG-02D3, Y1 ECS-320-12-37B2-7KM-TR, Y2 NX3215SA-32.768K-EXS00A-MU000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

Commit message: Remove additional spaces in Manufacturer_Part_Number field
Parts:
- C1, C3, C5, C7, C9: Manufacturer_Part_Number GRM155R71A104MA01D -> GRM155R71A104MA01D
- R1, R2, R3, R4: Manufacturer_Part_Number RC0402JR-0710KP -> RC0402JR-0710KP
Changed lines of the file:
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@@
 			)
 		)
-		(property "Manufacturer_Part_Number" "GRM155R71A104MA01D "
+		(property "Manufacturer_Part_Number" "GRM155R71A104MA01D"
 			(at 140.97 88.9 0)
 			(effects
@@
 			)
 		)
-		(property "Manufacturer_Part_Number" "GRM155R71A104MA01D "
+		(property "Manufacturer_Part_Number" "GRM155R71A104MA01D"
 			(at 69.85 109.22 0)
 			(effects
@@
 			)
 		)
-		(property "Manufacturer_Part_Number" "GRM155R71A104MA01D "
+		(property "Manufacturer_Part_Number" "GRM155R71A104MA01D"
 			(at 105.41 41.91 0)
 			(effects
@@
 			)
 		)
-		(property "Manufacturer_Part_Number" " RC0402JR-0710KP"
+		(property "Manufacturer_Part_Number" "RC0402JR-0710KP"
 			(at 106.68 66.04 0)
 			(effects
@@
 			)
 		)
-		(property "Manufacturer_Part_Number" "GRM155R71A104MA01D "
+		(property "Manufacturer_Part_Number" "GRM155R71A104MA01D"
 			(at 115.57 46.99 0)
 			(effects
@@
 			)
 		)
-		(property "Manufacturer_Part_Number" " RC0402JR-0710KP"
+		(property "Manufacturer_Part_Number" "RC0402JR-0710KP"
 			(at 100.33 52.07 0)
 			(effects
@@
 			)
 		)
-		(property "Manufacturer_Part_Number" " RC0402JR-0710KP"
+		(property "Manufacturer_Part_Number" "RC0402JR-0710KP"
 			(at 57.15 104.14 0)
 			(effects
@@
 			)
 		)
-		(property "Manufacturer_Part_Number" "GRM155R71A104MA01D "
+		(property "Manufacturer_Part_Number" "GRM155R71A104MA01D"
 			(at 137.16 109.22 0)
 			(effects
@@
 			)
 		)
-		(property "Manufacturer_Part_Number" " RC0402JR-0710KP"
+		(property "Manufacturer_Part_Number" "RC0402JR-0710KP"
 			(at 92.71 138.43 0)
 			(effects
