File: power_monitor.kicad_sch (KiCad schematic)
At the start: 6 parts, among them IC17 INA186A5IYFDR

Commit message: Add company name (using github URL), date, and change revision number to all schematic pages
Other:
- company: (none) -> github.com/fuad1502/open-running-watch-hw
Changed lines of the file:
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@@
 	(title_block
 		(title "Open Running Watch")
-		(rev "A")
+		(date "2024-04-12")
+		(rev "0.1.0")
+		(company "github.com/fuad1502/open-running-watch-hw")
 	)
 	(junction

Commit message: Changed hand soldered footprints to normal footprints
Parts:
- C72: footprint Capacitor_SMD:C_0402_1005Metric_Pad0.74x0.62mm_HandSolder -> Capacitor_SMD:C_0402_1005Metric
- R34: footprint Resistor_SMD:R_1206_3216Metric_Pad1.30x1.75mm_HandSolder -> Resistor_SMD:R_1206_3216Metric
- R35: footprint Resistor_SMD:R_0402_1005Metric_Pad0.72x0.64mm_HandSolder -> Resistor_SMD:R_0402_1005Metric
Changed lines of the file:
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@@
 			)
 		)
-		(property "Footprint" "Capacitor_SMD:C_0402_1005Metric_Pad0.74x0.62mm_HandSolder"
+		(property "Footprint" "Capacitor_SMD:C_0402_1005Metric"
 			(at 120.9548 105.41 0)
 			(effects
@@
 			)
 		)
-		(property "Footprint" "Resistor_SMD:R_1206_3216Metric_Pad1.30x1.75mm_HandSolder"
+		(property "Footprint" "Resistor_SMD:R_1206_3216Metric"
 			(at 146.05 93.218 90)
 			(effects
@@
 			)
 		)
-		(property "Footprint" "Resistor_SMD:R_0402_1005Metric_Pad0.72x0.64mm_HandSolder"
+		(property "Footprint" "Resistor_SMD:R_0402_1005Metric"
 			(at 169.672 104.14 90)
 			(effects
