File: power_monitor.kicad_sch (KiCad schematic)
At the start: 6 parts, among them IC17 INA186A5IYFDR

Commit message: Remove additional spaces in Manufacturer_Part_Number field
Parts:
- C72: Manufacturer_Part_Number GRM155R71A104MA01D -> GRM155R71A104MA01D
- R35: Manufacturer_Part_Number RC0402JR-0710KP -> RC0402JR-0710KP
Changed lines of the file:
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@@
 			)
 		)
-		(property "Manufacturer_Part_Number" "GRM155R71A104MA01D "
+		(property "Manufacturer_Part_Number" "GRM155R71A104MA01D"
 			(at 121.92 109.22 0)
 			(effects
@@
 			)
 		)
-		(property "Manufacturer_Part_Number" " RC0402JR-0710KP"
+		(property "Manufacturer_Part_Number" "RC0402JR-0710KP"
 			(at 171.45 104.14 0)
 			(effects
