File: power_monitor.kicad_sch (KiCad schematic)
At the start: 6 parts, among them IC17 INA186A5IYFDR

Commit message: Set 'do not populate' on power monitor probe point
Parts:
- TP6: now not fitted
Changed lines of the file:
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@@
 		(in_bom yes)
 		(on_board yes)
-		(dnp no)
+		(dnp yes)
 		(fields_autoplaced yes)
 		(property "Reference" "TP6"

Commit message: Upgrade to KiCad 10
Parts:
- renumbered IC17 to IC14, TP6 to TP1
