File: accelerometer.kicad_sch (KiCad schematic)
At the start: 5 parts

Commit message: Add company name (using github URL), date, and change revision number to all schematic pages
Other:
- company: (none) -> github.com/fuad1502/open-running-watch-hw
Changed lines of the file:
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@@
 	(title_block
 		(title "Open Running Watch")
-		(rev "A")
+		(date "2024-04-12")
+		(rev "0.1.0")
+		(company "github.com/fuad1502/open-running-watch-hw")
 	)
 	(junction

Commit message: Changed hand soldered footprints to normal footprints
Parts:
- C38, C39: footprint Capacitor_SMD:C_0402_1005Metric_Pad0.74x0.62mm_HandSolder -> Capacitor_SMD:C_0402_1005Metric
- C40, C41: footprint Capacitor_SMD:C_0603_1608Metric_Pad1.08x0.95mm_HandSolder -> Capacitor_SMD:C_0603_1608Metric
Changed lines of the file:
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@@
 			)
 		)
-		(property "Footprint" "Capacitor_SMD:C_0603_1608Metric_Pad1.08x0.95mm_HandSolder"
+		(property "Footprint" "Capacitor_SMD:C_0603_1608Metric"
 			(at 185.1152 105.41 0)
 			(effects
@@
 			)
 		)
-		(property "Footprint" "Capacitor_SMD:C_0603_1608Metric_Pad1.08x0.95mm_HandSolder"
+		(property "Footprint" "Capacitor_SMD:C_0603_1608Metric"
 			(at 188.9252 107.95 0)
 			(effects
@@
 			)
 		)
-		(property "Footprint" "Capacitor_SMD:C_0402_1005Metric_Pad0.74x0.62mm_HandSolder"
+		(property "Footprint" "Capacitor_SMD:C_0402_1005Metric"
 			(at 177.4952 107.95 0)
 			(effects
@@
 			)
 		)
-		(property "Footprint" "Capacitor_SMD:C_0402_1005Metric_Pad0.74x0.62mm_HandSolder"
+		(property "Footprint" "Capacitor_SMD:C_0402_1005Metric"
 			(at 173.6852 105.41 0)
 			(effects

Commit message: Remove additional spaces in Manufacturer_Part_Number field
Parts:
- C38, C39: Manufacturer_Part_Number GRM155R71A104MA01D -> GRM155R71A104MA01D
Changed lines of the file:
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@@
 			)
 		)
-		(property "Manufacturer_Part_Number" "GRM155R71A104MA01D "
+		(property "Manufacturer_Part_Number" "GRM155R71A104MA01D"
 			(at 176.53 111.76 0)
 			(effects
@@
 			)
 		)
-		(property "Manufacturer_Part_Number" "GRM155R71A104MA01D "
+		(property "Manufacturer_Part_Number" "GRM155R71A104MA01D"
 			(at 172.72 101.6 0)
 			(effects
