File: barometer.kicad_sch (KiCad schematic)
At the start: 2 parts, among them IC9 ICP-10100

Commit message: Add company name (using github URL), date, and change revision number to all schematic pages
Other:
- company: (none) -> github.com/fuad1502/open-running-watch-hw
Changed lines of the file:
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@@
 	(title_block
 		(title "Open Running Watch")
-		(rev "A")
+		(date "2024-04-12")
+		(rev "0.1.0")
+		(company "github.com/fuad1502/open-running-watch-hw")
 	)
 	(junction

Commit message: Changed hand soldered footprints to normal footprints
Parts:
- C42: footprint Capacitor_SMD:C_0402_1005Metric_Pad0.74x0.62mm_HandSolder -> Capacitor_SMD:C_0402_1005Metric
Changed lines of the file:
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@@
 			)
 		)
-		(property "Footprint" "Capacitor_SMD:C_0402_1005Metric_Pad0.74x0.62mm_HandSolder"
+		(property "Footprint" "Capacitor_SMD:C_0402_1005Metric"
 			(at 146.05 80.3148 0)
 			(effects

Commit message: Remove additional spaces in Manufacturer_Part_Number field
Parts:
- C42: Manufacturer_Part_Number GRM155R71A104MA01D -> GRM155R71A104MA01D
Changed lines of the file:
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@@
 			)
 		)
-		(property "Manufacturer_Part_Number" "GRM155R71A104MA01D "
+		(property "Manufacturer_Part_Number" "GRM155R71A104MA01D"
 			(at 142.24 81.28 0)
 			(effects
