File: gps.kicad_sch (KiCad schematic)
At the start: 14 parts, among them IC2 TESEO-LIV3F, IC3 BGA_725L6_E6327

Commit message: Remove additional spaces in Manufacturer_Part_Number field
Parts:
- C17, C18: Manufacturer_Part_Number GRM155R71A104MA01D -> GRM155R71A104MA01D
- C19, C21: Manufacturer_Part_Number GCM1555C1H121JA16D -> GCM1555C1H121JA16D
- FL1: Description_1 Frequency RF SAW Filter (Surface Acoustic Wave) Bandwidth 5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 -> (none)
- L3: Manufacturer_Part_Number LQW15AN5N6G80D -> LQW15AN5N6G80D
- R5: Manufacturer_Part_Number RC0402JR-0710KP -> RC0402JR-0710KP
