File: gps.kicad_sch (KiCad schematic)
At the start: 14 parts, among them IC2 TESEO-LIV3F, IC3 BGA_725L6_E6327

Commit message: Upgrade to KiCad 10
Changed lines of the file:
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@@
 (kicad_sch
-	(version 20231120)
+	(version 20260306)
 	(generator "eeschema")
-	(generator_version "8.0")
+	(generator_version "10.0")
 	(paper "A4")
 	(title_block
