File: power.kicad_sch (KiCad schematic)
At the start: 31 parts, among them IC13 TPS613222ADBVR, IC4 BQ27441DRZR-G1A, IC5 MCP73811T-420I_OT, IC6 TPS62237DRYR, IC7 ST1S15J18R, U1 TPS62233DRYR

Commit message: Changed regulator footprint to KiCad provided one
Parts:
- IC6: footprint TPS62237DRYR:TPS62237DRYR -> Package_SON:Texas_USON-6_1x1.45mm_P0.5mm_SMD
Changed lines of the file:
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@@
 			)
 		)
-		(property "Footprint" "TPS62237DRYR:TPS62237DRYR"
+		(property "Footprint" "Package_SON:Texas_USON-6_1x1.45mm_P0.5mm_SMD"
 			(at 165.1 178.74 0)
 			(effects

Commit message: Remove additional spaces in Manufacturer_Part_Number field
Parts:
- L6: Manufacturer_Part_Number LQM21PNR47MC0D -> LQM21PNR47MC0D
- L7: Manufacturer_Part_Number DFE252012F-2R2M=P2 -> DFE252012F-2R2M=P2
- R10, R11, R8: Manufacturer_Part_Number RC0402JR-0710KP -> RC0402JR-0710KP
- R9: Manufacturer_Part_Number RC0402JR-071ML -> RC0402JR-071ML
Changed lines of the file:
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@@
 			)
 		)
-		(property "Manufacturer_Part_Number" " RC0402JR-0710KP"
+		(property "Manufacturer_Part_Number" "RC0402JR-0710KP"
 			(at 171.45 55.88 0)
 			(effects
@@
 			)
 		)
-		(property "Manufacturer_Part_Number" "RC0402JR-071ML "
+		(property "Manufacturer_Part_Number" "RC0402JR-071ML"
 			(at 154.94 113.03 90)
 			(effects
@@
 			)
 		)
-		(property "Manufacturer_Part_Number" "DFE252012F-2R2M=P2 "
+		(property "Manufacturer_Part_Number" "DFE252012F-2R2M=P2"
 			(at 205.74 127 90)
 			(effects
@@
 			)
 		)
-		(property "Manufacturer_Part_Number" "LQM21PNR47MC0D "
+		(property "Manufacturer_Part_Number" "LQM21PNR47MC0D"
 			(at 154.94 139.7 90)
 			(effects
@@
 			)
 		)
-		(property "Manufacturer_Part_Number" " RC0402JR-0710KP"
+		(property "Manufacturer_Part_Number" "RC0402JR-0710KP"
 			(at 106.68 87.63 0)
 			(effects
@@
 			)
 		)
-		(property "Manufacturer_Part_Number" " RC0402JR-0710KP"
+		(property "Manufacturer_Part_Number" "RC0402JR-0710KP"
 			(at 171.45 90.17 0)
 			(effects

Commit message: Changed battery connection footprint
Parts:
- BT1: footprint Connector_Wire:SolderWire-0.1sqmm_1x02_P3.6mm_D0.4mm_OD1mm_Relief -> Connector_Wire:SolderWire-0.1sqmm_1x02_P3.6mm_D0.4mm_OD1mm
Changed lines of the file:
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@@
 			)
 		)
-		(property "Footprint" "Connector_Wire:SolderWire-0.1sqmm_1x02_P3.6mm_D0.4mm_OD1mm_Relief"
+		(property "Footprint" "Connector_Wire:SolderWire-0.1sqmm_1x02_P3.6mm_D0.4mm_OD1mm"
 			(at 35.56 133.096 90)
 			(effects
