File: open-running-watch.kicad_sch (KiCad schematic)
At the start: 0 parts

Commit message: TEMP COMMIT
Parts:
- added J10, J7, J8, J9: Conn_02x10_Odd_Even, Connector_PinHeader_2.54mm:PinHeader_2x10_P2.54mm_Vertical_SMD, symbol Connector_Generic:Conn_02x10_Odd_Even
Connections:
- new net BT_RESET_N: J9.13 (Pin_13)
- new net BT_SPI_CLK: J9.9 (Pin_9)
- new net BT_SPI_CS: J9.8 (Pin_8)
- new net BT_SPI_IN: J9.11 (Pin_11)
- new net BT_SPI_IRQ: J9.12 (Pin_12)
- new net BT_SPI_OUT: J9.10 (Pin_10)
- new net GPS_PPS: J9.5 (Pin_5)
- new net GPS_RESET_N: J9.7 (Pin_7)
- new net GPS_RX: J9.4 (Pin_4)
- new net GPS_TX: J9.3 (Pin_3)
- new net GPS_WAKEUP: J9.6 (Pin_6)
- new net MCU_3V3_EN: J7.1 (Pin_1)
- new net MCU_3V_EN: J7.2 (Pin_2)
- new net MCU_ACC_IRQ_1: J7.19 (Pin_19)
- new net MCU_ACC_IRQ_2: J7.18 (Pin_18)
- new net MCU_ADC_IN1: J8.4 (Pin_4)
- new net MCU_ADC_IN2: J8.5 (Pin_5)
- new net MCU_BT_IRQ: J7.12 (Pin_12)
- new net MCU_BT_RESET_N: J7.13 (Pin_13)
- new net MCU_FUEL_LOW: J8.13 (Pin_13)
- new net MCU_GPS_PPS: J7.5 (Pin_5)
- new net MCU_GPS_RESET_N: J7.7 (Pin_7)
- new net MCU_GPS_WAKEUP: J7.6 (Pin_6)
- new net MCU_HR_LED_G_1: J8.1 (Pin_1)
- new net MCU_HR_LED_G_2: J8.2 (Pin_2)
- new net MCU_HR_LED_IR: J8.3 (Pin_3)
- new net MCU_HR_LED_R: J7.20 (Pin_20)
- new net MCU_HR_OUT_IR_EN: J8.7 (Pin_7)
- new net MCU_HR_OUT_RG_EN: J8.6 (Pin_6)
- new net MCU_I2C_SCL: J8.12 (Pin_12), J8.9 (Pin_9)
- new net MCU_I2C_SDA: J8.11 (Pin_11), J8.8 (Pin_8)
- new net MCU_PWM: J8.10 (Pin_10)
- new net MCU_SPI_CS_1: J7.14 (Pin_14)
- new net MCU_SPI_CS_2: J7.8 (Pin_8)
- new net MCU_SPI_MISO: J7.10 (Pin_10), J7.16 (Pin_16)
- new net MCU_SPI_MOSI: J7.11 (Pin_11), J7.17 (Pin_17)
- new net MCU_SPI_SCL: J7.15 (Pin_15), J7.9 (Pin_9)
- new net MCU_USART_RX: J7.3 (Pin_3)
- new net MCU_USART_TX: J7.4 (Pin_4)
- new net PWR_3V3_EN: J9.1 (Pin_1)
- new net PWR_3V_EN: J9.2 (Pin_2)
- new net PWR_FUEL_LOW: J10.13 (Pin_13)
- new net PWR_FUEL_SCL: J10.12 (Pin_12)
- new net PWR_FUEL_SDA: J10.11 (Pin_11)
- new net SENS_CS: J9.14 (Pin_14)
- new net SENS_IN: J10.10 (Pin_10)
- new net SENS_INT_1: J9.19 (Pin_19)
- new net SENS_INT_2: J9.18 (Pin_18)
- new net SENS_IN_G1: J10.1 (Pin_1)
- new net SENS_IN_G2: J10.2 (Pin_2)
- new net SENS_IN_IR: J10.3 (Pin_3)
- new net SENS_IN_R: J9.20 (Pin_20)
- new net SENS_OUT_IR_EN: J10.7 (Pin_7)
- new net SENS_OUT_RG_EN: J10.6 (Pin_6)
- new net SENS_SCL: J10.9 (Pin_9)
- new net SENS_SDA: J10.8 (Pin_8)
- new net SENS_SDIO: J9.17 (Pin_17)
- new net SENS_SDO: J9.16 (Pin_16)
- new net SENS_SPC: J9.15 (Pin_15)
- new net SENS_VOUT_IR: J10.5 (Pin_5)
- new net SENS_VOUT_RG: J10.4 (Pin_4)
- no-connect marks 0 -> 14
Other:
- added sheet connectors (connectors.kicad_sch)
